File: esphome-denj/esphome-denj.kicad_sch (KiCad schematic)
At the start: 20 parts

Commit message: Denj V2 Schematic
Parts:
- removed Q?: IRFR2905Z, PCM_Package_TO_SOT_SMD_AKL:TO-252-2, symbol PCM_Transistor_MOSFET_AKL:IRFR2905Z
- removed R? (x3): 1k, Resistor_THT:R_Axial_DIN0207_L6.3mm_D2.5mm_P10.16mm_Horizontal, symbol PCM_SL_Resistors:1k
- added DZ? (x5): BZV48-C3V3, PCM_Diode_THT_AKL:D_DO-27_P15.24mm_Horizontal_Zener, symbol PCM_Diode_Zener_AKL:BZV48-C3V3
- added J? (x2): Conn_01x04, 4ms_Connector:Pins_1x04_2.54mm_TH_SWD, symbol PCM_4ms_Connector:Conn_01x04
- added J?: Screw_Terminal_01x08, symbol Connector:Screw_Terminal_01x08
- added J?: Conn_01x06, symbol Connector_Generic:Conn_01x06
- added J?: Screw_Terminal_2_P5.00mm, TerminalBlock_Phoenix:TerminalBlock_Phoenix_PT-1,5-2-5.0-H_1x02_P5.00mm_Horizontal, symbol PCM_SL_Screw_Terminal:Screw_Terminal_2_P5.00mm
- added Q? (x2): IRFR2905Z, PCM_Package_TO_SOT_SMD_AKL:TO-252-2, symbol PCM_Transistor_MOSFET_AKL:IRFR2905Z
- added Q?: BC547A, PCM_Package_TO_SOT_THT_AKL:TO-92_Inline_Wide_CBE, symbol PCM_Transistor_BJT_AKL:BC547A
- added R? (x7): 4.7k, Resistor_THT:R_Axial_DIN0207_L6.3mm_D2.5mm_P10.16mm_Horizontal, symbol PCM_SL_Resistors:1k
- added R? (x6): 1k, Resistor_THT:R_Axial_DIN0207_L6.3mm_D2.5mm_P10.16mm_Horizontal, symbol PCM_SL_Resistors:1k
- added U?: DS18B20, Package_TO_SOT_THT:TO-92_Inline, symbol Sensor_Temperature:DS18B20
- C? (x3): value 100nF_Ceramic -> 100nF
- R?: value 1k -> 24k
Connections:
- net +12V: now also J?.1, J?.1 (Pin_1), J?.2 (Pin_2)
- net +3.3V: now also J?.2 (Pin_2), J?.2 (Pin_2), J?.5 (Pin_5), R?.1, R?.1, R?.1, R?.1, U?.3 (V_{DD})
- net +5V: now also R?.2, R?.2
- net GND: now also J?.4, DZ?.2 (A), DZ?.2 (A), DZ?.2 (A), DZ?.2 (A), DZ?.2 (A), J?.1 (Pin_1), J?.1 (Pin_1), J?.2 (Pin_2), J?.3 (Pin_3), J?.5 (Pin_5), J?.6 (Pin_6), J?.8 (Pin_8), Q?.3 (E), Q?.3 (S), Q?.3 (S), R?.2, R?.2, U?.1 (GND); no longer J?.2
- net AC_HEATER: now reaches A?.7 (D6/GPIO12/MISO), R?.1
- net at Q?.2 (B): now also R?.2
- net DC_FAN: now reaches A?.8 (D5/GPIO14/SCLK)
- net DC_FAN: now also R?.1, R?.1
- net AC_LED: now reaches A?.6 (D7/GPIO13/MOSI/RX2)
- net AC_LED: now also R?.1
- net SDA: now reaches A?.13 (D2/GPIO4/SDA)
- net SDA: now also DZ?.1 (K), J?.4 (Pin_4), J?.4 (Pin_4), J?.7 (Pin_7), R?.2
- net SCL: now reaches A?.14 (D1/GPIO5/SCL)
- net SCL: now also DZ?.1 (K), J?.3 (Pin_3), J?.3 (Pin_3), J?.6 (Pin_6), R?.2
- net SW: now reaches A?.15 (D0/GPIO16/WAKE)
- net SW: now also DZ?.1 (K), J?.1 (Pin_1), R?.2
- net TACHO: now reaches A?.3 (GPIO1/TX0)
- net TACHO: now also DZ?.1 (K), R?.2
- net PWM: now reaches A?.4 (GPIO3/RX0)
- net PWM: now also R?.1
- net DC_LED: now reaches A?.5 (D8/GPIO15/CS/TX2)
- net DC_LED: now also R?.1, R?.1
- net Onboard_Button renamed BTN
- net Onboard_LED renamed 1W
- net 1W: now also DZ?.1 (K), J?.4 (Pin_4), R?.2, U?.2 (DQ)
- new net: Q?.1 (G), R?.2 (x2)
- new net: J?.2, Q?.2 (D) (x2)
- new net: J?.3 (Pin_3), R?.1, R?.1
- new net: J?.4 (Pin_4), Q?.1 (C), R?.1
- new net: Q?.2 (B), R?.2
Other:
- note added: "1-Wire"
- note added: "1W"
- note added: "3.3V"
- note added: "AC HEATER"
- note added: "AC IN"
- note added: "AC LED"
- note added: "DC FAN Filter"
- note added: "DC FAN Ventil"
- note added: "DC IN"
- note added: "DC LED"
- note added: "Door SW"
- note added: "GND"
- note added: "GND_Out_2"
- note added: "I2C"
- note added: "OLED"
- note added: "SCL"
- note added: "SDA"
- note added: "SW"
- note removed: "LED Internal"
- note removed: "LED Table"
- moved on the sheet: A?, C?, J?, K?, Q?, R?, U?

Commit message: Day 1008 Rev B
Parts:
- removed DZ? (x2): BZV48-C3V3, PCM_Diode_THT_AKL:D_DO-27_P15.24mm_Horizontal_Zener, symbol PCM_Diode_Zener_AKL:BZV48-C3V3
- removed J?: Conn_01x04, 4ms_Connector:Pins_1x04_2.54mm_TH_SWD, symbol PCM_4ms_Connector:Conn_01x04
- removed R? (x2): 4.7k, Resistor_THT:R_Axial_DIN0207_L6.3mm_D2.5mm_P10.16mm_Horizontal, symbol PCM_SL_Resistors:1k
- added C1, C2, C3, C4, C5: 220n, Capacitor_THT:C_Disc_D5.0mm_W2.5mm_P2.50mm, symbol PCM_SL_Capacitors:100nF_Ceramic
- added DZ4, DZ5: BZV48-C3V3, PCM_Diode_THT_AKL:D_DO-27_P15.24mm_Horizontal_Zener, symbol PCM_Diode_Zener_AKL:BZV48-C3V3
- added F1: Polyfuse_3A_15V, Fuse:Fuse_1812_4532Metric, symbol PCM_4ms_Regulator:Polyfuse_3A_15V
- added J1, J16, J3: Conn_01x04, 4ms_Connector:Pins_1x04_2.54mm_TH_SWD, symbol PCM_4ms_Connector:Conn_01x04
- added J10: Screw_Terminal_01x02, symbol Connector:Screw_Terminal_01x02
- added J14, J15, J7: PINHD_1x4_Female, Connector_PinSocket_2.54mm:PinSocket_1x04_P2.54mm_Vertical, symbol PCM_SL_Pin_Headers:PINHD_1x4_Female
- added J17: Screw_Terminal_01x03, symbol Connector:Screw_Terminal_01x03
- added J18: PINHD_1x3_Male, Connector_PinHeader_2.54mm:PinHeader_1x03_P2.54mm_Vertical, symbol PCM_SL_Pin_Headers:PINHD_1x3_Male
- added J19: Screw_Terminal_01x04, symbol Connector:Screw_Terminal_01x04
- added J6: PINHD_1x3_Female, Connector_PinSocket_2.54mm:PinSocket_1x03_P2.54mm_Vertical, symbol PCM_SL_Pin_Headers:PINHD_1x3_Female
- added R5, R6: 6.8k, Resistor_THT:R_Axial_DIN0207_L6.3mm_D2.5mm_P10.16mm_Horizontal, symbol PCM_SL_Resistors:1k
- added SW1: SW_Nidec_CAS-120A1, Button_Switch_SMD:Nidec_Copal_CAS-120A, symbol Switch:SW_Nidec_CAS-120A1
- added U2, U4: DS18B20, Package_TO_SOT_THT:TO-92_Inline, symbol Sensor_Temperature:DS18B20
- C6: renamed from C?; value 100nF -> 220n
- C7, C8: renamed from C?; value 100nF -> 330n
- R1, R2, R3, R4, R7: renamed from R?; value 4.7k -> 6.8k
- R10: renamed from R?; value 1k -> 1.5015k
- R11, R12, R8: renamed from R?; value 1k -> 6.8k
- R15: renamed from R?; value 1k -> 510
- R16: renamed from R?; value 1k -> 1.5k
- R9: renamed from R?; value 24k -> 47.436k
- gave numbers to parts that had none: 23
Connections:
- net +12V: now also J2.3 (Pin_3), J2.4 (Pin_4), C1.1, J3.2 (Pin_2); no longer J2.1 (Pin_1), J2.2 (Pin_2)
- net +3.3V: now also J4.4 (Pin_4), C3.1, C4.1, C5.1, F1.1, J1.2 (Pin_2), J6.1, J7.2, R5.1, R6.1; no longer A1.1 (3V3), A1.10 (3V3), A1.26 (3V3), J4.5 (Pin_5), U3.3 (V_{DD})
- net +5V: now also C2.1
- net 1W: now also J4.5 (Pin_5), J6.2; no longer J4.4 (Pin_4), U3.2 (DQ)
- net AC_L_1: no longer J11.1, K1.3
- net DC_FAN: now also R15.1, R16.1; no longer R11.1, R12.1
- net DC_LED: now also R11.1, R12.1; no longer R15.1, R16.1
- net GND: now also J2.1 (Pin_1), J2.2 (Pin_2), J4.1 (Pin_1), J4.6 (Pin_6), J4.7 (Pin_7), C1.2, C2.2, C3.2, C4.2, C5.2, DZ4.2 (A), DZ5.2 (A), J1.1 (Pin_1), J3.1 (Pin_1), J6.3, J7.1; no longer J2.5 (Pin_5), J2.6 (Pin_6), J4.2 (Pin_2), J4.3 (Pin_3), J4.8 (Pin_8), U3.1 (GND)
- net SCL: now also J4.3 (Pin_3), DZ4.1 (K), J1.3 (Pin_3), J7.3, R5.2; no longer J4.6 (Pin_6)
- net SDA: now also J4.2 (Pin_2), DZ5.1 (K), J1.4 (Pin_4), J7.4, R6.2; no longer J4.7 (Pin_7)
- net SW: now also J4.8 (Pin_8); no longer J4.1 (Pin_1)
- net at R2.1, R7.1: now also J2.5 (Pin_5), J3.3 (Pin_3); no longer J2.3 (Pin_3)
- net at Q1.1 (C), R1.1: now also J2.6 (Pin_6), J3.4 (Pin_4); no longer J2.4 (Pin_4)
- new net: J17.1 (Pin_1), U2.3 (V_{DD}), U3.3 (V_{DD})
- new net: J17.2 (Pin_2), U2.2 (DQ), U3.2 (DQ)
- new net: J17.3 (Pin_3), U2.1 (GND), U3.1 (GND)
- new net: J18.3, U4.1 (GND)
- new net: J18.2, U4.2 (DQ)
- new net: J18.1, U4.3 (V_{DD})
- new net: J11.1, K1.3
- new net: J10.1 (Pin_1), SW1.1 (C)
- new net: J10.2 (Pin_2), SW1.2 (B)
- new net: A1.1 (3V3), A1.10 (3V3), A1.26 (3V3), F1.2
- new net BME280/GND: J14.1
- new net BME280/SCL: J14.3
- new net BME280/SDA: J14.4
- new net BME280/VCC: J14.2
- new net Keyboard/GND: J19.1 (Pin_1)
- new net Keyboard/SCL: J19.3 (Pin_3)
- new net Keyboard/SDA: J19.2 (Pin_2)
- new net Keyboard/VCC: J19.4 (Pin_4)
- new net OLED SSD1306/GND: J16.1 (Pin_1)
- new net OLED SSD1306/SCL: J16.3 (Pin_3)
- new net OLED SSD1306/SDA: J16.4 (Pin_4)
- new net OLED SSD1306/VCC: J16.2 (Pin_2)
- new net RTC DS3231/GND: J15.1
- new net RTC DS3231/SCL: J15.3
- new net RTC DS3231/SDA: J15.4
- new net RTC DS3231/VCC: J15.2
Other:
- added sheet BME280 (bme280.kicad_sch)
- added sheet Keyboard (keyboard.kicad_sch)
- added sheet OLED SSD1306 (oled.kicad_sch)
- added sheet RTC DS3231 (rtc.kicad_sch)
- note added: "1-W"
- note added: "HV"
- note added: "I2C BME280"
- note added: "I2C OLED"
- note added: "I2C RTC"
- note added: "OPTIONAL"
- note added: "PWM"
- note added: "TACH"
- note removed: "Door SW"
- note removed: "OLED"
- company: (none) -> avatarsd LLC
- title: (none) -> SLA-BOX
- moved on the sheet: A1, C6, C7, C8, DZ1, DZ2, DZ3, J11, J12, J13, J2, J4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
